File: PCB/01-main/01-main.sch (EAGLE design)
At the start: 64 parts, among them CN1 ML8, J1 22057045, J14 22057055, J8 22057045, Q1 C1015, SW1 SK-12D11VG3, T1 BSS138, U1 CH340ESMD, U2 STM32F446RET6, U3 SUNA_LIB_M5STAMP_C3U_MATE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

Commit message: ⚡️基礎配線完了
Connections:
- removed net N$22: R10.2, U1.TNOW
- removed net N$23: LED18.A, R10.1
- new net N$19: LED18.A, U1.TNOW
- new net N$20: LED18.C, R10.2
- net GND: now also R10.1; no longer J14.3, LED18.C
- net LED-FLOOR: no longer CN1.6
- net MIRROR: no longer CN1.8
- net SIG-FLOOR: no longer CN1.5
- net TOGGLE: now also CN1.8
- net UART3-RX: now also CN1.5
- net UART3-TX: now also CN1.6
- net UART4-TX: now also J14.3
Other:
- moved on the sheet: LED18, R10
Changed lines of the file:
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@@
 <attribute name="VALUE" x="45.72" y="78.74" size="1.778" layer="96"/>
 </instance>
-<instance part="R10" gate="G$1" x="58.42" y="53.34" smashed="yes" rot="R180">
-<attribute name="NAME" x="53.34" y="55.88" size="1.778" layer="95"/>
-<attribute name="VALUE" x="53.34" y="48.26" size="1.778" layer="96"/>
-</instance>
-<instance part="LED18" gate="G$1" x="68.58" y="53.34" smashed="yes" rot="R90">
-<attribute name="NAME" x="66.04" y="55.88" size="1.778" layer="95"/>
-<attribute name="VALUE" x="66.04" y="47.244" size="1.778" layer="96"/>
+<instance part="R10" gate="G$1" x="73.66" y="53.34" smashed="yes" rot="R180">
+<attribute name="NAME" x="68.58" y="55.88" size="1.778" layer="95"/>
+<attribute name="VALUE" x="68.58" y="48.26" size="1.778" layer="96"/>
+</instance>
+<instance part="LED18" gate="G$1" x="58.42" y="53.34" smashed="yes" rot="R90">
+<attribute name="NAME" x="55.88" y="55.88" size="1.778" layer="95"/>
+<attribute name="VALUE" x="55.88" y="47.244" size="1.778" layer="96"/>
 </instance>
 <instance part="GND44" gate="1" x="81.28" y="48.26" smashed="yes">
@@
 </segment>
 <segment>
-<pinref part="LED18" gate="G$1" pin="C"/>
-<wire x1="73.66" y1="53.34" x2="81.28" y2="53.34" width="0.1524" layer="91"/>
 <wire x1="81.28" y1="53.34" x2="81.28" y2="50.8" width="0.1524" layer="91"/>
 <pinref part="GND44" gate="1" pin="GND"/>
+<pinref part="R10" gate="G$1" pin="1"/>
+<wire x1="78.74" y1="53.34" x2="81.28" y2="53.34" width="0.1524" layer="91"/>
 </segment>
 <segment>
@@
 </segment>
 </net>
-<net name="N$22" class="0">
-<segment>
-<pinref part="U1" gate="G$1" pin="TNOW"/>
-<wire x1="50.8" y1="53.34" x2="53.34" y2="53.34" width="0.1524" layer="91"/>
-<pinref part="R10" gate="G$1" pin="2"/>
-</segment>
-</net>
-<net name="N$23" class="0">
-<segment>
-<pinref part="R10" gate="G$1" pin="1"/>
-<wire x1="63.5" y1="53.34" x2="66.04" y2="53.34" width="0.1524" layer="91"/>
-<pinref part="LED18" gate="G$1" pin="A"/>
-</segment>
-</net>
 <net name="UART1-TX" class="0">
 <segment>
@@
 <wire x1="124.46" y1="99.06" x2="116.84" y2="99.06" width="0.1524" layer="91"/>
 <label x="101.6" y="99.06" size="1.778" layer="95"/>
+</segment>
+</net>
+<net name="N$19" class="0">
+<segment>
+<pinref part="LED18" gate="G$1" pin="A"/>
+<pinref part="U1" gate="G$1" pin="TNOW"/>
+<wire x1="55.88" y1="53.34" x2="50.8" y2="53.34" width="0.1524" layer="91"/>
+</segment>
+</net>
+<net name="N$20" class="0">
+<segment>
+<pinref part="R10" gate="G$1" pin="2"/>
+<pinref part="LED18" gate="G$1" pin="C"/>
+<wire x1="68.58" y1="53.34" x2="63.5" y2="53.34" width="0.1524" layer="91"/>
 </segment>
 </net>
@@
 <wire x1="210.82" y1="58.46" x2="210.82" y2="58.42" width="0.1524" layer="91"/>
 <wire x1="210.82" y1="58.42" x2="218.44" y2="58.42" width="0.1524" layer="91"/>
-<wire x1="218.44" y1="58.42" x2="218.44" y2="55.88" width="0.1524" layer="91"/>
 <pinref part="GND35" gate="1" pin="GND"/>
 <pinref part="J14" gate="A" pin="2"/>
-<pinref part="J14" gate="A" pin="3"/>
-<wire x1="218.44" y1="55.88" x2="218.44" y2="48.26" width="0.1524" layer="91"/>
-<wire x1="210.82" y1="55.88" x2="218.44" y2="55.88" width="0.1524" layer="91"/>
-<junction x="218.44" y="55.88"/>
+<wire x1="218.44" y1="58.42" x2="218.44" y2="48.26" width="0.1524" layer="91"/>
 </segment>
 <segment>
@@
 <wire x1="40.64" y1="149.86" x2="38.1" y2="149.86" width="0.1524" layer="91"/>
 <label x="27.94" y="149.86" size="1.778" layer="95"/>
+</segment>
+</net>
+<net name="UART4-TX" class="0">
+<segment>
+<pinref part="J14" gate="A" pin="3"/>
+<wire x1="210.82" y1="55.88" x2="220.98" y2="55.88" width="0.1524" layer="91"/>
+<label x="223.52" y="55.88" size="1.778" layer="95"/>
 </segment>
 </net>
@@
 <label x="101.6" y="157.48" size="1.778" layer="95"/>
 </segment>
+<segment>
+<pinref part="CN1" gate="1" pin="8"/>
+<wire x1="215.9" y1="53.34" x2="226.06" y2="53.34" width="0.1524" layer="91"/>
+<label x="228.6" y="53.34" size="1.778" layer="95"/>
+</segment>
 </net>
 <net name="+3V3" class="0">
@@
 </segment>
 </net>
-<net name="LED-FLOOR" class="0">
+<net name="SERVO-SIG" class="0">
+<segment>
+<pinref part="CN1" gate="1" pin="7"/>
+<wire x1="208.28" y1="53.34" x2="198.12" y2="53.34" width="0.1524" layer="91"/>
+<label x="180.34" y="53.34" size="1.778" layer="95"/>
+</segment>
+</net>
+<net name="UART1-TX" class="0">
+<segment>
+<wire x1="231.14" y1="160.02" x2="238.76" y2="160.02" width="0.1524" layer="91"/>
+<label x="241.3" y="160.02" size="1.778" layer="95"/>
+<pinref part="U3" gate="G$1" pin="G20"/>
+</segment>
+</net>
+<net name="UART3-RX" class="0">
+<segment>
+<pinref part="CN1" gate="1" pin="5"/>
+<wire x1="208.28" y1="55.88" x2="198.12" y2="55.88" width="0.1524" layer="91"/>
+<label x="180.34" y="55.88" size="1.778" layer="95"/>
+</segment>
+</net>
+<net name="UART3-TX" class="0">
 <segment>
 <wire x1="215.9" y1="55.88" x2="226.06" y2="55.88" width="0.1524" layer="91"/>
@@
 </segment>
 </net>
-<net name="SERVO-SIG" class="0">
-<segment>
-<pinref part="CN1" gate="1" pin="7"/>
-<wire x1="208.28" y1="53.34" x2="198.12" y2="53.34" width="0.1524" layer="91"/>
-<label x="180.34" y="53.34" size="1.778" layer="95"/>
-</segment>
-</net>
-<net name="MIRROR" class="0">
-<segment>
-<pinref part="CN1" gate="1" pin="8"/>
-<wire x1="215.9" y1="53.34" x2="226.06" y2="53.34" width="0.1524" layer="91"/>
-<label x="228.6" y="53.34" size="1.778" layer="95"/>
-</segment>
-</net>
-<net name="SIG-FLOOR" class="0">
-<segment>
-<pinref part="CN1" gate="1" pin="5"/>
-<wire x1="208.28" y1="55.88" x2="198.12" y2="55.88" width="0.1524" layer="91"/>
-<label x="180.34" y="55.88" size="1.778" layer="95"/>
-</segment>
-</net>
-<net name="UART1-TX" class="0">
-<segment>
-<wire x1="231.14" y1="160.02" x2="238.76" y2="160.02" width="0.1524" layer="91"/>
-<label x="241.3" y="160.02" size="1.778" layer="95"/>
-<pinref part="U3" gate="G$1" pin="G20"/>
-</segment>
-</net>

Commit message: ⚡️ ERC
Parts:
- added J2, J3: 22057025, con-molex-5268:22057025
Connections:
- removed net LED-FLOOR: U2A.PB15
- removed net LED-UI: U2A.PB14
- removed net MIRROR: U2A.PA11
- removed net SIG-FLOOR: U2A.PC0
- removed net SWCLK: U2A.PA14
- removed net SWDIO: U2A.PA13
- new net CAM-LED-L: J3.2, U2A.PB15
- new net CAM-LED-R: J2.2, U2A.PB14
- net GND: now also J2.1, J3.1
Other:
- note added: "BLE"
- note added: "BOTTOM"
- note added: "LED"
- note removed: "XIAO"
- moved on the sheet: C13, C16, C7, C8, C9, CN1, D1, R30, R31, R4, REG1, S1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
