File: PCB/03-LiDAR/03-LiDAR.brd (EAGLE design)
At the start: 80 x 93 mm, 57 parts, among them U2 PCA9555PW,112

Commit message: ✨ 基本配線完了
Parts:
- added C16, C18, C6, C7, C8, C9: 0.1µ, rcl:C0603
- added C5: 4.7µ, rcl:C0603
- added JP1: (no value), pinhead:1X04
- added LED21, LED22: WHITE, led:SML0603
- added R15, R16: 5k1, rcl:R0402
- added R18, R32: 270, rcl:R0402
- added R30, R31: 10k, rcl:R0402
- added SW1: SK-12D11VG3, Slide Switch:SK-12D11VG3
- added TP6, TP8, TP9: PTR1TP10R, testpad:TP10R
- added TP7: PTR1TP10SQ, testpad:TP10SQ
- added U3: STM32F446RET6, F446RE:LQFP64-10X10MM
- added U4: CH340ESMD, CH340E:MSOP10
- added X2: usb-c, microbuilder:USB_C_CUSB31-CFM2AX-01-X
- moved R10 4.16 mm to (26.7, -3.81)
- moved C1 4.00 mm to (6.00, 6.00)
- moved C2 4.00 mm to (6.00, -2.00)
- moved C3 4.00 mm to (12.0, 9.00)
- moved C4 4.00 mm to (12.0, -5.00)
- moved D1 4.00 mm to (4.00, 2.00)
- moved REG1 4.00 mm to (12.0, 2.00)
- moved TP1 3.00 mm to (2.54, -23.8)
- moved TP2 3.00 mm to (1.27, -23.8)
- moved TP3 3.00 mm to (0.00, -23.8)
- moved TP4 3.00 mm to (-1.27, -23.8)
- moved TP5 3.00 mm to (-2.54, -23.8)
Connections:
- removed net RX: TP3.TP, U1.8
- removed net TX: TP4.TP, U1.7
- new net BOOT0: R31.1, SW1.1, U3.60
- new net CTS: U4.5
- new net D+: U4.1, X2.A6, X2.B6
- new net D-: U4.2, X2.A7, X2.B7
- new net LED-WHITE: LED22.A, U3.33
- new net LIDAR_PWM: TP8.TP, U3.22
- new net N$17: R15.1, X2.A5
- new net N$18: R16.1, X2.B5
- new net N$20: C5.1, U3.30
- new net N$21: C16.1, U4.10
- new net N$22: LED21.A, U4.6
- new net N$26: LED21.C, R18.2
- new net N$32: LED22.C, R32.2
- new net NRST: C18.1, R30.2, U3.7
- new net RTS: U4.4
- new net SWO: U3.55
- new net UART1-RX: U3.43, U4.8
- new net UART1-TX: U3.42, U4.9
- new net UART2-RX: TP9.TP, U3.17
- new net UART2-TX: U3.16
- new net UART4-RX: U1.7, U3.15
- new net UART4-TX: U3.14
- new net UART5-RX: TP3.TP, U1.8, U3.54
- new net UART5-TX: TP4.TP, U3.53
- new net VBUS: X2.A4B9, X2.B4A9
- net +3V3: now also C6.1, C7.1, C8.1, C9.1, JP1.3, R30.1, SW1.3, U3.1, U3.13, U3.19, U3.32, U3.48, U3.64
- net +5V: now also TP6.TP, U4.7
- net GND: now also C16.2, C18.2, C5.2, C6.2, C7.2, C8.2, C9.2, JP1.4, R15.2, R16.2, R18.1, R31.2, R32.1, SW1.4, SW1.5, TP7.TP, U3.12, U3.18, U3.31, U3.47, U3.63, U4.3, X2.A1B12, X2.B1A12
- net SCL: now also JP1.2
- net SDA: now also JP1.1
Routing:
- net GND: track 238.3 -> 443.9 mm, vias 0 -> 3
- net +3V3: track 80.9 -> 217.3 mm, vias 0 -> 3
- net LED_SIG: track 0.00 -> 66.7 mm, vias 0 -> 2
- net SDA: track 145.7 -> 205.5 mm, vias 0 -> 1
- net +5V: track 188.9 -> 245.3 mm, vias 0 -> 3
- net N$9: track 0.00 -> 55.9 mm
- net SCL: track 147.2 -> 201.5 mm, vias 0 -> 2
- net BOOT0: track 0.00 -> 37.6 mm
- net UART4-RX: track 0.00 -> 28.9 mm
- net UART5-RX: track 0.00 -> 25.1 mm, vias 0 -> 2
- net VDD: track 14.0 -> 37.1 mm, vias 0 -> 1
- net LED-WHITE: track 0.00 -> 22.8 mm, vias 0 -> 2
- net LIDAR_PWM: track 0.00 -> 19.6 mm
- net UART1-TX: track 0.00 -> 17.3 mm
- net UART1-RX: track 0.00 -> 17.3 mm
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Other:
- outline, holes or cut-outs redrawn

Commit message: ✨ とりあえずできた、一晩寝かせる
Parts:
- moved JP1 0.70 mm to (0.00, -50.1)
Routing:
- net GND: track 443.9 -> 643.7 mm
- net +3V3: track 217.3 -> 373.6 mm, vias 3 -> 7
- net +5V: track 245.3 -> 286.3 mm, vias 3 -> 4
- net X5: track 2.13 -> 36.0 mm, vias 0 -> 1
- net X6: track 9.04 -> 40.6 mm, vias 0 -> 1
- net X4: track 2.46 -> 31.2 mm, vias 0 -> 1
- net X7: track 2.47 -> 28.7 mm, vias 0 -> 1
- net X8: track 2.43 -> 25.9 mm, vias 0 -> 1
- net X3: track 2.43 -> 23.8 mm, vias 0 -> 2
- net X9: track 2.47 -> 21.0 mm, vias 0 -> 1
- net X2: track 2.47 -> 19.1 mm, vias 0 -> 1
- net X1: track 2.43 -> 12.0 mm
- net SCL: track 201.5 -> 200.8 mm
Other:
- outline, holes or cut-outs redrawn

Commit message: ✨ LiDARのシルク入れ完了
Routing:
- net GND: vias 3 -> 16
- added copper zone on layer 1, net GND
- added copper zone on layer 16, net GND
Other:
- board text added: "/Users/shirokuma89dev/Downloads/アートボード 1@4x.bmp"
- board text added: "/Users/shirokuma89dev/Downloads/アートボード 2@4x (1).bmp"
