File: PCB/02-PWR/02-PWR.sch (EAGLE design)
At the start: 67 parts, among them CN1 ML8-R, J1 5267-3, J2 5267-3, J3 5267-3, J4 5267-3, J5 22057045, J6 22057045, J7 5267-3, J8 5267-3, J9 3557-2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

Commit message: ✨エンコーダー配線完了
Parts:
- added C10, C6, C9: 0.1µ, rcl:C-EUC0603
- added JP7, JP8: (no value), pinhead:PINHD-1X5
- added R20, R21, R22, R23, R24, R25: 10k, rcl:R-EU_R0402
Connections:
- new net ENC_A: C9.1, R22.1, U2A.PA14
- new net ENC_B: C6.1, R21.2, U2A.PA15
- new net ENC_SW: C10.1, JP8.3, R25.1, U2A.PB7
- new net LED_B: JP8.4, U2A.PB6
- new net LED_G: JP8.2, U2A.PB5
- new net LED_R: R20.2, U2A.PB4
- new net N$21: JP7.4, R21.1, R24.2
- new net N$22: JP7.2, R22.2, R23.2
- new net N$23: JP8.1, R20.1
- net +3V3: now also JP8.5, R23.1, R24.1
- net GND: now also C10.2, C6.2, C9.2, JP7.3, R25.2
- net XSHUT1: now also U2A.PA5
- net XSHUT2: now also U2A.PA6
Other:
- moved on the sheet: C11, C17, CN1, D2, J1, J2, J3, J4, J7, J8, J9, REG2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

Commit message: ✨ 下段完成
Parts:
- added TP1, TP2: PTR1TP16R, testpad:PTR1TP16R
Connections:
- net GND: now also TP2.TP
- net VDD: now also TP1.TP
Changed lines of the file:
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@@
 <setting verticaltext="up"/>
 </settings>
-<grid distance="0.1" unitdist="inch" unit="inch" style="lines" multiple="1" display="yes" altdistance="0.01" altunitdist="inch" altunit="inch"/>
+<grid distance="0.1" unitdist="inch" unit="inch" style="lines" multiple="1" display="no" altdistance="0.01" altunitdist="inch" altunit="inch"/>
 <layers>
 <layer number="1" name="Top" color="4" fill="1" visible="no" active="no"/>
@@
 <part name="R22" library="rcl" library_urn="urn:adsk.eagle:library:334" deviceset="R-EU_" device="R0402" package3d_urn="urn:adsk.eagle:package:23547/3" value="10k"/>
 <part name="R20" library="rcl" library_urn="urn:adsk.eagle:library:334" deviceset="R-EU_" device="R0402" package3d_urn="urn:adsk.eagle:package:23547/3" value="10k"/>
+<part name="TP1" library="testpad" library_urn="urn:adsk.eagle:library:385" deviceset="PTR1" device="TP16R" package3d_urn="urn:adsk.eagle:package:27969/1"/>
+<part name="TP2" library="testpad" library_urn="urn:adsk.eagle:library:385" deviceset="PTR1" device="TP16R" package3d_urn="urn:adsk.eagle:package:27969/1"/>
+<part name="VDD9" library="supply1" library_urn="urn:adsk.eagle:library:371" deviceset="VDD" device=""/>
+<part name="GND41" library="supply1" library_urn="urn:adsk.eagle:library:371" deviceset="GND" device=""/>
 </parts>
 <sheets>
@@
 <attribute name="VALUE" x="101.6" y="-55.88" size="1.778" layer="96"/>
 </instance>
+<instance part="TP1" gate="G$1" x="175.26" y="149.86" smashed="yes" rot="R270">
+<attribute name="NAME" x="168.91" y="150.876" size="1.778" layer="95"/>
+<attribute name="TP_SIGNAL_NAME" x="172.72" y="148.59" size="1.778" layer="97" rot="R270"/>
+</instance>
+<instance part="TP2" gate="G$1" x="175.26" y="144.78" smashed="yes" rot="R270">
+<attribute name="NAME" x="168.91" y="145.796" size="1.778" layer="95"/>
+<attribute name="TP_SIGNAL_NAME" x="172.72" y="143.51" size="1.778" layer="97" rot="R270"/>
+</instance>
+<instance part="VDD9" gate="G$1" x="180.34" y="154.94" smashed="yes">
+<attribute name="VALUE" x="182.88" y="152.4" size="1.778" layer="96"/>
+</instance>
+<instance part="GND41" gate="1" x="180.34" y="139.7" smashed="yes">
+<attribute name="VALUE" x="177.8" y="137.16" size="1.778" layer="96"/>
+</instance>
 </instances>
 <busses>
@@
 <pinref part="GND40" gate="1" pin="GND"/>
 </segment>
+<segment>
+<pinref part="GND41" gate="1" pin="GND"/>
+<pinref part="TP2" gate="G$1" pin="TP"/>
+<wire x1="180.34" y1="142.24" x2="180.34" y2="144.78" width="0.1524" layer="91"/>
+<wire x1="180.34" y1="144.78" x2="177.8" y2="144.78" width="0.1524" layer="91"/>
+</segment>
 </net>
 <net name="VDD" class="0">
@@
 <wire x1="195.58" y1="129.54" x2="195.58" y2="132.08" width="0.1524" layer="91"/>
 </segment>
+<segment>
+<pinref part="TP1" gate="G$1" pin="TP"/>
+<wire x1="177.8" y1="149.86" x2="180.34" y2="149.86" width="0.1524" layer="91"/>
+<wire x1="180.34" y1="149.86" x2="180.34" y2="152.4" width="0.1524" layer="91"/>
+<pinref part="VDD9" gate="G$1" pin="VDD"/>
+</segment>
 </net>

Commit message: ♻️ 再配線中
Parts:
- removed S1: (no value), switch-omron:31-XX
- J5, J6: value 22057045 -> 5267-4; device con-molex-5268:22057045 -> con-molex-spox:5267-4
Connections:
- net +3V3: now also J5.-1, J6.-1; no longer J5.1, J6.1
- net GND: now also J5.-2, J6.-2; no longer J5.2, J6.2, S1.S
- net N$1: now also J5.-3; no longer J5.3
- net N$2: now also J5.-4; no longer J5.4
- net N$5: now also J6.-3; no longer J6.3
- net N$6: now also J6.-4; no longer J6.4
- net NRST: no longer S1.P
Changed lines of the file:
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@@
 <part name="+3V2" library="supply1" library_urn="urn:adsk.eagle:library:371" deviceset="+3V3" device=""/>
 <part name="GND10" library="supply1" library_urn="urn:adsk.eagle:library:371" deviceset="GND" device=""/>
-<part name="J5" library="con-molex-5268" deviceset="22057045" device=""/>
 <part name="+3V4" library="supply1" library_urn="urn:adsk.eagle:library:371" deviceset="+3V3" device=""/>
 <part name="GND12" library="supply1" library_urn="urn:adsk.eagle:library:371" deviceset="GND" device=""/>
@@
 <part name="R4" library="rcl" library_urn="urn:adsk.eagle:library:334" deviceset="R-EU_" device="R0805" package3d_urn="urn:adsk.eagle:package:23553/2" value="330k"/>
 <part name="GND14" library="supply1" library_urn="urn:adsk.eagle:library:371" deviceset="GND" device=""/>
-<part name="J6" library="con-molex-5268" deviceset="22057045" device=""/>
 <part name="+3V6" library="supply1" library_urn="urn:adsk.eagle:library:371" deviceset="+3V3" device=""/>
 <part name="GND15" library="supply1" library_urn="urn:adsk.eagle:library:371" deviceset="GND" device=""/>
@@
 <part name="JP5" library="pinhead" library_urn="urn:adsk.eagle:library:325" deviceset="PINHD-2X4" device="" package3d_urn="urn:adsk.eagle:package:22461/2"/>
 <part name="JP6" library="pinhead" library_urn="urn:adsk.eagle:library:325" deviceset="PINHD-2X4" device="" package3d_urn="urn:adsk.eagle:package:22461/2"/>
-<part name="S1" library="switch-omron" library_urn="urn:adsk.eagle:library:377" deviceset="31-XX" device="" package3d_urn="urn:adsk.eagle:package:27487/1"/>
-<part name="GND50" library="supply1" library_urn="urn:adsk.eagle:library:371" deviceset="GND" device=""/>
 <part name="R30" library="rcl" library_urn="urn:adsk.eagle:library:334" deviceset="R-EU_" device="R0402" package3d_urn="urn:adsk.eagle:package:23547/3" value="10k"/>
 <part name="+3V15" library="supply1" library_urn="urn:adsk.eagle:library:371" deviceset="+3V3" device=""/>
@@
 <part name="VDD9" library="supply1" library_urn="urn:adsk.eagle:library:371" deviceset="VDD" device=""/>
 <part name="GND41" library="supply1" library_urn="urn:adsk.eagle:library:371" deviceset="GND" device=""/>
+<part name="J5" library="con-molex-spox" deviceset="5267-4" device=""/>
+<part name="J6" library="con-molex-spox" deviceset="5267-4" device=""/>
 </parts>
 <sheets>
@@
 <attribute name="VALUE" x="510.54" y="154.94" size="1.778" layer="96"/>
 </instance>
-<instance part="J5" gate="A" x="20.32" y="81.28" smashed="yes" rot="MR0">
-<attribute name="NAME" x="16.1544" y="86.5886" size="2.0828" layer="95" ratio="6" rot="SMR0"/>
-</instance>
 <instance part="+3V4" gate="G$1" x="25.4" y="86.36" smashed="yes">
 <attribute name="VALUE" x="27.94" y="83.82" size="1.778" layer="96"/>
@@
 <instance part="GND14" gate="1" x="68.58" y="86.36" smashed="yes">
 <attribute name="VALUE" x="66.04" y="83.82" size="1.778" layer="96"/>
-</instance>
-<instance part="J6" gate="A" x="20.32" y="35.56" smashed="yes" rot="MR0">
-<attribute name="NAME" x="16.1544" y="40.8686" size="2.0828" layer="95" ratio="6" rot="SMR0"/>
 </instance>
 <instance part="+3V6" gate="G$1" x="25.4" y="40.64" smashed="yes">
@@
 <attribute name="VALUE" x="494.03" y="83.82" size="1.778" layer="96"/>
 </instance>
-<instance part="S1" gate="1" x="393.7" y="157.48" smashed="yes" rot="R270">
-<attribute name="NAME" x="391.795" y="163.83" size="1.778" layer="95"/>
-<attribute name="VALUE" x="396.875" y="161.29" size="1.778" layer="96"/>
-</instance>
-<instance part="GND50" gate="1" x="401.32" y="152.4" smashed="yes">
-<attribute name="VALUE" x="398.78" y="149.86" size="1.778" layer="96"/>
-</instance>
 <instance part="R30" gate="G$1" x="383.54" y="165.1" smashed="yes" rot="R270">
 <attribute name="NAME" x="375.92" y="165.1" size="1.778" layer="95"/>
@@
 <instance part="GND41" gate="1" x="180.34" y="139.7" smashed="yes">
 <attribute name="VALUE" x="177.8" y="137.16" size="1.778" layer="96"/>
+</instance>
+<instance part="J5" gate="G$1" x="20.32" y="78.74" smashed="yes" rot="MR0">
+<attribute name="VALUE" x="20.32" y="70.74" size="1.27" layer="94" rot="MR0"/>
+<attribute name="NAME" x="20.32" y="83.88" size="1.27" layer="94" rot="MR0"/>
+</instance>
+<instance part="J6" gate="G$1" x="20.32" y="33.02" smashed="yes" rot="MR0">
+<attribute name="VALUE" x="20.32" y="25.02" size="1.27" layer="94" rot="MR0"/>
+<attribute name="NAME" x="20.32" y="38.16" size="1.27" layer="94" rot="MR0"/>
 </instance>
 </instances>
@@
 </segment>
 <segment>
-<pinref part="J5" gate="A" pin="2"/>
 <wire x1="20.32" y1="78.74" x2="25.4" y2="78.74" width="0.1524" layer="91"/>
 <wire x1="25.4" y1="78.74" x2="25.4" y2="71.12" width="0.1524" layer="91"/>
 <pinref part="GND12" gate="1" pin="GND"/>
+<pinref part="J5" gate="G$1" pin="-2"/>
 </segment>
 <segment>
@@
 </segment>
 <segment>
-<pinref part="J6" gate="A" pin="2"/>
 <wire x1="20.32" y1="33.02" x2="25.4" y2="33.02" width="0.1524" layer="91"/>
 <wire x1="25.4" y1="33.02" x2="25.4" y2="25.4" width="0.1524" layer="91"/>
 <pinref part="GND15" gate="1" pin="GND"/>
+<pinref part="J6" gate="G$1" pin="-2"/>
 </segment>
 <segment>
@@
 </segment>
 <segment>
-<pinref part="GND50" gate="1" pin="GND"/>
-<pinref part="S1" gate="1" pin="S"/>
-<wire x1="398.78" y1="157.48" x2="401.32" y2="157.48" width="0.1524" layer="91"/>
-<wire x1="401.32" y1="154.94" x2="401.32" y2="157.48" width="0.1524" layer="91"/>
-</segment>
-<segment>
 <pinref part="GND51" gate="1" pin="GND"/>
 <pinref part="C16" gate="G$1" pin="2"/>
@@
 </segment>
 <segment>
-<pinref part="J5" gate="A" pin="1"/>
 <wire x1="20.32" y1="81.28" x2="25.4" y2="81.28" width="0.1524" layer="91"/>
 <wire x1="25.4" y1="81.28" x2="25.4" y2="83.82" width="0.1524" layer="91"/>
 <pinref part="+3V4" gate="G$1" pin="+3V3"/>
+<pinref part="J5" gate="G$1" pin="-1"/>
 </segment>
 <segment>
@@
 </segment>
 <segment>
-<pinref part="J6" gate="A" pin="1"/>
 <wire x1="20.32" y1="35.56" x2="25.4" y2="35.56" width="0.1524" layer="91"/>
 <wire x1="25.4" y1="35.56" x2="25.4" y2="38.1" width="0.1524" layer="91"/>
 <pinref part="+3V6" gate="G$1" pin="+3V3"/>
+<pinref part="J6" gate="G$1" pin="-1"/>
 </segment>
 <segment>
@@
 <net name="N$1" class="0">
 <segment>
-<pinref part="J5" gate="A" pin="3"/>
 <wire x1="20.32" y1="76.2" x2="27.94" y2="76.2" width="0.1524" layer="91"/>
 <wire x1="27.94" y1="76.2" x2="30.48" y2="73.66" width="0.1524" layer="91"/>
 <pinref part="R2" gate="G$1" pin="1"/>
 <wire x1="30.48" y1="73.66" x2="33.02" y2="73.66" width="0.1524" layer="91"/>
+<pinref part="J5" gate="G$1" pin="-3"/>
 </segment>
 </net>
@@
 <pinref part="R1" gate="G$1" pin="1"/>
 <wire x1="33.02" y1="78.74" x2="27.94" y2="73.66" width="0.1524" layer="91"/>
-<pinref part="J5" gate="A" pin="4"/>
 <wire x1="27.94" y1="73.66" x2="20.32" y2="73.66" width="0.1524" layer="91"/>
+<pinref part="J5" gate="G$1" pin="-4"/>
 </segment>
 </net>
@@
 <net name="N$5" class="0">
 <segment>
-<pinref part="J6" gate="A" pin="3"/>
 <wire x1="20.32" y1="30.48" x2="27.94" y2="30.48" width="0.1524" layer="91"/>
 <wire x1="27.94" y1="30.48" x2="30.48" y2="27.94" width="0.1524" layer="91"/>
 <pinref part="R6" gate="G$1" pin="1"/>
 <wire x1="30.48" y1="27.94" x2="33.02" y2="27.94" width="0.1524" layer="91"/>
+<pinref part="J6" gate="G$1" pin="-3"/>
 </segment>
 </net>
@@
 <pinref part="R5" gate="G$1" pin="1"/>
 <wire x1="33.02" y1="33.02" x2="27.94" y2="27.94" width="0.1524" layer="91"/>
-<pinref part="J6" gate="A" pin="4"/>
 <wire x1="27.94" y1="27.94" x2="20.32" y2="27.94" width="0.1524" layer="91"/>
+<pinref part="J6" gate="G$1" pin="-4"/>
 </segment>
 </net>
@@
 </segment>
 <segment>
-<pinref part="S1" gate="1" pin="P"/>
-<wire x1="388.62" y1="157.48" x2="383.54" y2="157.48" width="0.1524" layer="91"/>
 <label x="363.22" y="157.48" size="1.778" layer="95"/>
 <pinref part="R30" gate="G$1" pin="2"/>
@@
 <wire x1="381" y1="157.48" x2="373.38" y2="157.48" width="0.1524" layer="91"/>
 <wire x1="383.54" y1="157.48" x2="383.54" y2="160.02" width="0.1524" layer="91"/>
-<junction x="383.54" y="157.48"/>
 <pinref part="C16" gate="G$1" pin="1"/>
 <wire x1="381" y1="154.94" x2="381" y2="157.48" width="0.1524" layer="91"/>
