File: PCB/02-PWR/02-PWR.brd (EAGLE design)
At the start: 88 x 158.5 mm, 67 parts, among them CN1 ML8-R, J1 5267-3, J2 5267-3, J3 5267-3, J4 5267-3, J5 22057045, J6 22057045, J7 5267-3, J8 5267-3, J9 3557-2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

Commit message: ✨エンコーダー配線完了
Parts:
- added C10, C6, C9: 0.1µ, rcl:C0603
- added JP7, JP8: (no value), pinhead:1X05
- added R20, R21, R22, R23, R24, R25: 10k, rcl:R0402
Connections:
- new net ENC_A: C9.1, R22.1, U2.49
- new net ENC_B: C6.1, R21.2, U2.50
- new net ENC_SW: C10.1, JP8.3, R25.1, U2.59
- new net LED_B: JP8.4, U2.58
- new net LED_G: JP8.2, U2.57
- new net LED_R: R20.2, U2.56
- new net N$21: JP7.4, R21.1, R24.2
- new net N$22: JP7.2, R22.2, R23.2
- new net N$23: JP8.1, R20.1
- net +3V3: now also JP8.5, R23.1, R24.1
- net GND: now also C10.2, C6.2, C9.2, JP7.3, R25.2
- net XSHUT1: now also U2.21
- net XSHUT2: now also U2.22
Routing:
- net +3V3: track 25.4 -> 379.4 mm, vias 0 -> 9
- net GND: track 360.3 -> 703.1 mm, vias 8 -> 14
- net LED-WHITE: track 0.00 -> 127.9 mm, vias 0 -> 2
- net NRST: track 4.44 -> 85.8 mm, vias 0 -> 1
- net XSHUT1: track 0.00 -> 74.9 mm, vias 0 -> 3
- net XSHUT2: track 0.00 -> 63.3 mm, vias 0 -> 2
- net +5V: track 64.7 -> 124.8 mm, vias 0 -> 2
- net KIT_R: track 0.00 -> 58.6 mm, vias 0 -> 1
- net KIT_L: track 0.00 -> 51.9 mm, vias 0 -> 1
- net ENC_A: track 0.00 -> 51.9 mm, vias 0 -> 2
- net BOOT0: track 0.00 -> 44.7 mm
- net N$19: track 0.00 -> 35.8 mm, vias 0 -> 2
- net ENC_SW: track 0.00 -> 34.8 mm, vias 0 -> 1
- net LED_G: track 0.00 -> 33.2 mm, vias 0 -> 1
- net SDA: track 65.7 -> 98.7 mm
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
Commit message: ✨ 下段完成
Parts:
- added TP1, TP2: PTR1TP16R, testpad:TP16R
Connections:
- net GND: now also TP2.TP
- net VDD: now also TP1.TP
Routing:
- net VDD: track 247.0 -> 304.7 mm
- net TOGGLE_LED: track 25.7 -> 28.5 mm, vias 1 -> 2
- net GND: vias 14 -> 65
- added copper zone on layer 1, net GND
- added copper zone on layer 16, net GND

Commit message: ♻️ 再配線中
Parts:
- removed S1: (no value), switch-omron:B3F-31XX
- J5, J6: value 22057045 -> 5267-4; device con-molex-5268:CON_22057045_MOL -> con-molex-spox:5267-4
- moved C11 43.0 mm to (-4.00, 33.0)
- moved C17 43.0 mm to (4.00, 33.0)
- moved D2 43.0 mm to (0.00, 30.0)
- moved REG2 43.0 mm to (0.00, 37.0)
- moved SW3 8.51 mm to (4.00, -72.0)
- moved U3 6.40 mm to (-5.00, -70.0)
- moved AMP1 6.00 mm to (-5.00, 46.5)
- moved AMP2 6.00 mm to (5.00, 46.5)
- moved R3 6.00 mm to (-2.00, 47.0)
- moved R4 6.00 mm to (-8.00, 47.0)
- moved R7 6.00 mm to (8.00, 47.0)
- moved R8 6.00 mm to (2.00, 47.0)
- moved J5 5.02 mm to (-11.0, 62.0), turned to 0 degrees
- moved J6 5.02 mm to (3.50, 62.0), turned to 0 degrees
- moved R19 4.00 mm to (-6.00, 69.0)
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Connections:
- net +3V3: now also J5.P$1, J6.P$1; no longer J5.1, J6.1
- net GND: now also J5.P$2, J6.P$2; no longer J5.2, J6.2, S1.2
- net N$1: now also J5.P$3; no longer J5.3
- net N$2: now also J5.P$4; no longer J5.4
- net N$5: now also J6.P$3; no longer J6.3
- net N$6: now also J6.P$4; no longer J6.4
- net NRST: no longer S1.1
Routing:
- net GND: track 703.1 -> 377.2 mm, vias 65 -> 9
- net +3V3: track 379.4 -> 76.5 mm, vias 9 -> 0
- net SERVO-SIG: track 257.7 -> 146.6 mm, vias 1 -> 2
- net +5V: track 124.8 -> 21.4 mm, vias 2 -> 0
- net NRST: track 85.8 -> 4.49 mm, vias 1 -> 0
- net XSHUT1: track 74.9 -> 0.00 mm, vias 3 -> 0
- net LED-WHITE: track 127.9 -> 62.4 mm, vias 2 -> 0
- net XSHUT2: track 63.3 -> 0.00 mm, vias 2 -> 0
- net KIT_R: track 58.6 -> 0.00 mm, vias 1 -> 0
- net KIT_L: track 51.9 -> 0.00 mm, vias 1 -> 0
- net MCU_RX-SUB_TX: track 48.6 -> 0.00 mm, vias 1 -> 0
- net VDD: track 304.7 -> 256.3 mm, vias 3 -> 9
- net MCU_TX-SUB_RX: track 41.1 -> 0.00 mm, vias 1 -> 0
- net TOGGLE: track 45.8 -> 5.12 mm, vias 1 -> 0
- net BOOT0: track 44.7 -> 4.59 mm
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- removed copper zone on layer 1, net GND
- removed copper zone on layer 16, net GND

Commit message: ♻️ ほぼ完成
Parts:
- moved C14 12.1 mm to (-7.00, -67.5), turned to 180 degrees
- turned LED17 to 270 degrees
Routing:
- net GND: track 377.2 -> 709.3 mm, vias 9 -> 14
- net +3V3: track 76.5 -> 261.1 mm, vias 0 -> 7
- net SERVO-SIG: track 146.6 -> 224.2 mm, vias 2 -> 3
- net XSHUT1: track 0.00 -> 67.7 mm, vias 0 -> 2
- net XSHUT2: track 0.00 -> 59.2 mm, vias 0 -> 2
- net VDD: track 256.3 -> 311.8 mm
- net MCU_RX-SUB_TX: track 0.00 -> 45.3 mm, vias 0 -> 1
- net BOOT0: track 4.59 -> 49.7 mm, vias 0 -> 1
- net MCU_TX-SUB_RX: track 0.00 -> 38.1 mm, vias 0 -> 1
- net TOGGLE: track 5.12 -> 40.6 mm, vias 0 -> 1
- net LOADCELL-R: track 38.7 -> 42.1 mm
- net LED-WHITE: track 62.4 -> 59.4 mm
- net N$11: track 0.00 -> 1.81 mm

Commit message: ✨ 完了
Routing:
- net +5V: track 21.4 -> 132.6 mm, vias 0 -> 2
- net GND: track 709.3 -> 806.9 mm, vias 14 -> 61
- net +3V3: track 261.1 -> 344.2 mm, vias 7 -> 10
- net LED-WHITE: track 59.4 -> 128.7 mm, vias 0 -> 4
- net KIT_R: track 0.00 -> 61.4 mm, vias 0 -> 3
- net KIT_L: track 0.00 -> 55.4 mm, vias 0 -> 1
- net N$10: track 20.1 -> 52.7 mm
- net TOGGLE_LED: track 23.8 -> 27.3 mm, vias 0 -> 1
- net TOGGLE: track 40.6 -> 43.2 mm, vias 1 -> 2
- net N$13: track 17.6 -> 15.7 mm
- net LED_B: track 26.8 -> 26.1 mm
- added copper zone on layer 1, net GND
- added copper zone on layer 16, net GND
